Commit message: spring fix

File: description/board/urdf/robot_core.xacro (robot description, xacro)
@@ -118,4 +118,5 @@
       effort="10"
       velocity="0.1" />
+<dynamics damping="0.5" friction="0.0"/>
   </joint>
   <link
@@ -285,4 +286,5 @@
       effort="10"
       velocity="0.1" />
+<dynamics damping="0.5" friction="0.0"/>
   </joint>
   <link
@@ -394,3 +396,11 @@
       xyz="0 -1 0" />
   </joint>
+<gazebo reference="trj0">
+  <springStiffness>0.5</springStiffness>
+  <springReference>0.0</springReference>
+</gazebo>
+<gazebo reference="trj1">
+  <springStiffness>0.5</springStiffness>
+  <springReference>0.0</springReference>
+</gazebo>
 </robot>

Commit message: test

File: description/board/urdf/robot_core.xacro (robot description, xacro)
@@ -113,10 +113,6 @@
     <axis
       xyz="0 0 -1" />
-    <limit
-      lower="-0.227799"
-      upper="0.227799"
-      effort="10"
-      velocity="0.1" />
-<!-- <dynamics damping="1.0" friction="0.1"/> -->
+    <limit lower="-0.227799" upper="0.227799" effort="50" velocity="1.0" />
+    <dynamics damping="0.5" friction="0.05"/>
   </joint>
   <link
@@ -281,10 +277,6 @@
     <axis
       xyz="0 0 -1" />
-    <limit
-      lower="-0.227799"
-      upper="0.227799"
-      effort="10"
-      velocity="0.1" />
-<!-- <dynamics damping="1.0" friction="0.1"/> -->
+    <limit lower="-0.227799" upper="0.227799" effort="50" velocity="1.0" />
+    <dynamics damping="0.5" friction="0.05"/>
   </joint>
   <link

File: description/board/urdf/ros2_control.xacro (robot description, xacro)
@@ -7,5 +7,5 @@
       </hardware>
       <!-- Truck joints (steering) -->
-      <joint name="trj0">
+      <!-- <joint name="trj0">
         <command_interface name="position">
           <param name="min">-0.227799</param>
@@ -25,4 +25,5 @@
         <state_interface name="effort"/>
       </joint>
+       -->
       <!-- Wheel joints -->
       <joint name="whj0">
