Commit message: test1

File: description/board/urdf/ros2_control.xacro (robot description, xacro)
@@ -6,24 +6,23 @@
         <plugin>gazebo_ros2_control/GazeboSystem</plugin>
       </hardware>
-      <!-- Truck joints (steering) -->
-      <!-- <joint name="trj0">
-        <command_interface name="position">
-          <param name="min">-0.227799</param>
-          <param name="max">0.227799</param>
-        </command_interface>
-        <state_interface name="position"/>
-        <state_interface name="velocity"/>
-        <state_interface name="effort"/>
-      </joint>
-      <joint name="trj1">
-        <command_interface name="position">
-          <param name="min">-0.227799</param>
-          <param name="max">0.227799</param>
-        </command_interface>
-        <state_interface name="position"/>
-        <state_interface name="velocity"/>
-        <state_interface name="effort"/>
-      </joint>
-       -->
+<!-- Truck joints (steering) -->
+<joint name="trj0">
+  <command_interface name="position">
+    <param name="min">-0.227799</param>
+    <param name="max">0.227799</param>
+  </command_interface>
+  <state_interface name="position"/>
+  <state_interface name="velocity"/>
+  <state_interface name="effort"/>
+</joint>
+<joint name="trj1">
+  <command_interface name="position">
+    <param name="min">-0.227799</param>
+    <param name="max">0.227799</param>
+  </command_interface>
+  <state_interface name="position"/>
+  <state_interface name="velocity"/>
+  <state_interface name="effort"/>
+</joint>
       <!-- Wheel joints -->
       <joint name="whj0">
