Commit message: fixed position topic

File: description/board/urdf/gazebo_control.xacro (robot description, xacro)
@@ -1,29 +1,11 @@
 <?xml version="1.0"?>
 <robot xmlns:xacro="http://www.ros.org/wiki/xacro">
-  <!-- Основной плагин для интеграции с ROS Control -->
+  <!-- Gazebo plugins -->
   <gazebo>
-    <plugin name="gazebo_ros_control" filename="libgazebo_ros_control.so">
-      <robotNamespace>/skate</robotNamespace>
-    </plugin>
-  </gazebo>
-  <!-- Публикатор состояний всех суставов -->
-  <gazebo>
-    <plugin name="joint_state_publisher" filename="libgazebo_ros_joint_state_publisher.so">
-      <jointName>trj0, trj1, whj0, whj1, whj2, whj3</jointName>
-      <updateRate>50.0</updateRate>
-      <robotNamespace>/skate</robotNamespace>
-    </plugin>
-  </gazebo>
-  <!-- Контроллеры для грузовиков (trj0, trj1) -->
-  <gazebo>
-    <plugin name="trj0_position_controller" filename="libgazebo_ros_joint_position_controller.so">
-      <jointName>trj0</jointName>
-      <robotNamespace>/skate</robotNamespace>
-    </plugin>
-  </gazebo>
-  <gazebo>
-    <plugin name="trj1_position_controller" filename="libgazebo_ros_joint_position_controller.so">
-      <jointName>trj1</jointName>
-      <robotNamespace>/skate</robotNamespace>
+    <!-- Joint state publisher -->
+    <plugin name="gazebo_ros_joint_state_publisher" filename="libgazebo_ros_joint_state_publisher.so">
+      <update_rate>20</update_rate>
+      <joint_name>trj0</joint_name>
+      <joint_name>trj1</joint_name>
     </plugin>
   </gazebo>

File: description/board/urdf/robot_core.xacro (robot description, xacro)
@@ -119,12 +119,4 @@
       velocity="0.1" />
   </joint>
-  <!-- Torsional Spring Plugin for trj0 -->
-  <gazebo>
-    <plugin name="trj0_torsional_spring" filename="libgazebo_joint_torsional_spring.so">
-      <kx>3.0</kx>
-      <set_point>0</set_point>
-      <joint>trj0</joint>
-    </plugin>
-  </gazebo>
   <link
     name="wh0">
@@ -294,12 +286,4 @@
       velocity="0.1" />
   </joint>
-  <!-- Torsional Spring Plugin for trj1 -->
-  <gazebo>
-    <plugin name="trj1_torsional_spring" filename="libgazebo_joint_torsional_spring.so">
-      <kx>3.0</kx>
-      <set_point>0</set_point>
-      <joint>trj1</joint>
-    </plugin>
-  </gazebo>
   <link
     name="wh2">

Commit message: odom

File: description/board/urdf/gazebo_control.xacro (robot description, xacro)
@@ -8,5 +8,40 @@
       <joint_name>trj0</joint_name>
       <joint_name>trj1</joint_name>
+      <!-- <joint_name>whj0</joint_name>
+      <joint_name>whj1</joint_name>
+      <joint_name>whj2</joint_name>
+      <joint_name>whj3</joint_name> -->
+    </plugin>
+    <!-- P3D position tracking plugin -->
+    <plugin name="skate_pos" filename="libgazebo_ros_p3d.so">
+      <body_name>base_link</body_name>
+      <frame_name>world</frame_name>
+      <update_rate>20.0</update_rate>
+      <xyz_offset>0 0 0</xyz_offset>
+      <rpy_offset>0 0 0</rpy_offset>
+      <!-- <gaussian_noise>0.01</gaussian_noise> -->
+      <topic>odom</topic>
     </plugin>
   </gazebo>
+  <!-- Add friction to the wheels for more realistic physics -->
+  <gazebo reference="wh0">
+    <mu1>0.8</mu1>
+    <mu2>0.8</mu2>
+    <material>Gazebo/Blue</material>
+  </gazebo>
+  <gazebo reference="wh1">
+    <mu1>0.8</mu1>
+    <mu2>0.8</mu2>
+    <material>Gazebo/Blue</material>
+  </gazebo>
+  <gazebo reference="wh2">
+    <mu1>0.8</mu1>
+    <mu2>0.8</mu2>
+    <material>Gazebo/Blue</material>
+  </gazebo>
+  <gazebo reference="wh3">
+    <mu1>0.8</mu1>
+    <mu2>0.8</mu2>
+    <material>Gazebo/Blue</material>
+  </gazebo>
 </robot>

Commit message: footlink added

File: description/board/urdf/gazebo_control.xacro (robot description, xacro)
@@ -22,5 +22,5 @@
     <!-- P3D position tracking plugin -->
     <plugin name="skate_pos" filename="libgazebo_ros_p3d.so">
-      <body_name>base_link</body_name>
+      <body_name>base_footprint</body_name>
       <frame_name>world</frame_name>
       <update_rate>20.0</update_rate>

File: description/board/urdf/robot_core.xacro (robot description, xacro)
@@ -13,10 +13,10 @@
 <color rgba="0 0 0 1"/>
 </material>
-<!-- <link name="base_footprint" />
+<link name="base_footprint" />
 <joint name="base_footprint_joint" type="fixed">
   <parent link="base_footprint" />
   <child link="base_link" />
   <origin xyz="0 0 0" rpy="0 0 0"/>
-</joint> -->
+</joint>
   <link
     name="base_link">
